File: pcb_kicad/wifitools/wifitools.kicad_pcb (KiCad board)
At the start: 2 copper layers, 4 parts

Commit message: Big update
Parts:
- removed the REF** at (137.2, 101.6)
- removed the REF** at (133.3, 152.8)
- removed the REF** at (158.8, 129.5)
- removed the REF** at (148.6, 78.7)
- added ?: LOGO, Lib:logo, F.Cu at (165.1, 68.6)
- added ?: LoLin V3 NodeMCU, ESP8266:NodeMCU-LoLinV3, B.Cu at (154.9, 106.7)
- added A: button 2pin, Lib:button, F.Cu at (160.0, 88.9)
- added B: button 2pin, Lib:button, F.Cu at (152.4, 99.1)
- added DOWN: button 2pin, Lib:button, F.Cu at (129.5, 99.1)
- added Display : Display, Lib:Display, F.Cu at (142.2, 63.5)
- added LEFT: button 2pin, Lib:button, F.Cu at (121.9, 94.0)
- added R1: Resistor, Lib:Resistor, B.Cu at (142.2, 139.7)
- added R2: Resistor, Lib:Resistor, B.Cu at (142.2, 144.8)
- added REF**: BatteryHolder_Keystone_1042_1x18650, Battery:BatteryHolder_Keystone_1042_1x18650, B.Cu at (124.5, 99.1)
- added RIGHT: button 2pin, Lib:button, F.Cu at (137.2, 94.0)
- added Senter: LED_D3.0mm_FlatTop, LED_THT:LED_D3.0mm_FlatTop, F.Cu at (167.6, 55.9)
- added UP: button 2pin, Lib:button, F.Cu at (129.5, 88.9)
Routing:
- net (no net): track 501.2 -> 904.2 mm
Other:
- board text added: "@Dx4Grey"
- board text added: "A"
- board text added: "B"
- board text added: "WiFi Tools"
