File: pcb-design/miaw-wifitools.kicad_pcb (KiCad board)
At the start: 2 copper layers, 30.5 x 60.3 mm, 19 parts

Commit message: Update PCBs
Parts:
- added G***: LOGO, WiFiTools:logo, F.Cu at (148.6, 95.2)
- 0.96 Oled SSD1306: renamed from ?
