File: WiFi Tik II/miaw-wifitools.kicad_pcb (KiCad board)
At the start: 2 copper layers, 45.7 x 60.3 mm, 24 parts

Commit message: Update
Parts:
- added G***: LOGO, WiFiTools:logo, F.Cu at (141.3, 76.8)
- moved display socket 3.87 mm to (152.4, 87.1)
- moved HOLE 3.39 mm to (138.9, 128.5)
- moved HOLE 3.39 mm to (138.9, 71.6)
- moved RX 3.39 mm to (131.4, 89.4)
- moved TX 3.39 mm to (131.4, 86.9)
- moved (D1 MINI) 3.39 mm to (152.4, 111.1)
- moved 0.96 Oled SSD1306 3.39 mm to (152.4, 81.3)
- moved B 3.39 mm to (153.9, 115.5)
- moved Battery 3.39 mm to (161.0, 74.2)
- moved DOWN 3.39 mm to (144.5, 115.5)
- moved G*** 3.39 mm to (133.3, 94.6)
- moved GPIO 0 3.39 mm to (168.9, 93.4)
- moved HOLE 3.39 mm to (165.8, 128.5)
- moved HOLE 3.39 mm to (165.8, 71.6)
- moved R1 3.39 mm to (146.0, 92.7)
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Routing:
- net /GND: track 456.4 -> 455.9 mm
Other:
- board text added: "dx4grey@github.io | ffffff | do you hate me? | i have all about you | Dx4 ft. Tantik"
- board text removed: "WiFiTik 2.0"
